Commit message: reorg assets

File: gym_solo/assets/solo8v2/solo.urdf (robot description, URDF)
Before this commit: robot solo, 13 links, 12 joints
Links:
- link FL_FOOT: geometry collision mesh filename=solo_foot.stl; visual mesh filename=solo_foot.stl
- link FL_LOWER_LEG: geometry collision mesh filename=solo_lower_leg_left_side.stl; visual mesh filename=solo_lower_leg_left_side.stl
- link FL_UPPER_LEG: geometry collision mesh filename=solo_upper_leg_left_side.stl; visual mesh filename=solo_upper_leg_left_side.stl
- link FR_FOOT: geometry collision mesh filename=solo_foot.stl; visual mesh filename=solo_foot.stl
- link FR_LOWER_LEG: geometry collision mesh filename=solo_lower_leg_right_side.stl; visual mesh filename=solo_lower_leg_right_side.stl
- link FR_UPPER_LEG: geometry collision mesh filename=solo_upper_leg_right_side.stl; visual mesh filename=solo_upper_leg_right_side.stl
- link HL_FOOT: geometry collision mesh filename=solo_foot.stl; visual mesh filename=solo_foot.stl
- link HL_LOWER_LEG: geometry collision mesh filename=solo_lower_leg_left_side.stl; visual mesh filename=solo_lower_leg_left_side.stl
- link HL_UPPER_LEG: geometry collision mesh filename=solo_upper_leg_left_side.stl; visual mesh filename=solo_upper_leg_left_side.stl
- link HR_FOOT: geometry collision mesh filename=solo_foot.stl; visual mesh filename=solo_foot.stl
- link HR_LOWER_LEG: geometry collision mesh filename=solo_lower_leg_right_side.stl; visual mesh filename=solo_lower_leg_right_side.stl
- link HR_UPPER_LEG: geometry collision mesh filename=solo_upper_leg_right_side.stl; visual mesh filename=solo_upper_leg_right_side.stl
- link base_link: geometry collision mesh filename=solo_body.stl; visual mesh filename=solo_body.stl
